File: Schematic/ClockProject.kicad_pcb (KiCad board)
At the start: 2 copper layers, 400 x 100 mm, 62 parts, among them J1 Conn_01x07_Pin, J10 Conn_01x03_Pin, J11 Conn_01x03_Pin, J13 Conn_01x03_Pin, J2 Conn_01x07_Pin, J3 Conn_01x07_Pin, J4 Conn_01x07_Pin, J5 Conn_01x09_Socket, J6 Conn_01x09_Socket, J9 USB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

Commit message: Fixed multiple initial issues
Fixed Silk for Connectors (GND move)
Fixed Boot/Reset Silk
Moved Edge Connectors closer to edge
Parts:
- moved J1 1.50 mm to (471.9, 180.6)
- moved J2 1.50 mm to (284.9, 143.6)
- moved J3 1.50 mm to (97.9, 180.6)
- moved J4 1.50 mm to (284.9, 217.6)
Routing:
- net +5V: track 858.5 -> 867.3 mm
- net /IC2: track 692.2 -> 699.9 mm
- net /IC3: track 698.1 -> 705.7 mm
- net /IC1: track 686.3 -> 693.9 mm
- net /U2: track 726.4 -> 734.0 mm
- net /U1: track 673.5 -> 680.8 mm
- net GND: track 552.3 -> 549.5 mm
Other:
- board text added: "Clock Module V1.1 Febuary 2025 Ian and Garrett Jordan"
- board text added: "U1 5V IC1 IC2 IC3 GND U2"
- board text removed: "Clock Module V1.0 Febuary 2025 Ian and Garrett Jordan"
- board text removed: "U1 5V GND IC1 IC2 IC3 U2"
